Commit message: Added box_spawn module

File: src/smart_palletizer_py/urdf/medium_box.urdf (robot description, URDF)
Before this commit: robot medium_box, 1 links, 0 joints
Links:
- removed link None
- added link base_link; visual box size=0.340 0.250 0.095

File: src/smart_palletizer_py/urdf/small_box.urdf (robot description, URDF)
Before this commit: robot small_box, 1 links, 0 joints
Links:
- removed link None
- added link base_link; visual box size=0.255 0.155 0.100
